Commit message: pitch joint에 마찰력 추가

File: urdf/gimbal.xacro (robot description, xacro)
@@ -32,7 +32,7 @@
   </link>
   <gazebo>
-    <plugin filename="libgz_ros2_control-system.so" name="gz_ros2_control::GazeboSimROS2ControlPlugin">
-      <parameters>$(find gimbal_demo)/config/controller.yaml</parameters>
-    </plugin>
+      <plugin filename="libgz_ros2_control-system.so" name="gz_ros2_control::GazeboSimROS2ControlPlugin">
+          <parameters>$(find gimbal_demo)/config/controller.yaml</parameters>
+      </plugin>
   </gazebo>
   <!-- yaw_link -->
@@ -114,4 +114,5 @@
     <origin xyz="0 0 0.05" rpy="0 0 0"/>
     <axis xyz="0 1 0"/>
+    <dynamics damping="0.7" friction="0.1"/>
     <limit lower="-1.57" upper="0.5" effort="5.0" velocity="2.0"/>
   </joint>

Commit message: 목표 위치 시각화 노드 추가 (구면좌표계 -> 직교 좌표계)

File: urdf/gimbal.xacro (robot description, xacro)
@@ -128,5 +128,5 @@
     <child link="camera_optical_frame"/>
     <!-- ROS 카메라 표준 REP-103 optical frame 변환 -->
-    <origin xyz="0 0 0" rpy="${-pi/2} 0 ${-pi/2}"/>
+    <origin xyz="0.02 0 0" rpy="${-pi/2} 0 ${-pi/2}"/>
   </joint>
   <!-- Gazebo 카메라 센서 -->
@@ -173,3 +173,60 @@
     </joint>
   </ros2_control>
+  <link name="tof_link">
+    <visual>
+      <geometry>
+        <box size="0.01 0.01 0.005"/>
+      </geometry>
+      <material name="black">
+        <color rgba="0 0 0 1"/>
+      </material>
+    </visual>
+    <collision>
+      <geometry>
+        <box size="0.01 0.01 0.005"/>
+      </geometry>
+    </collision>
+    <inertial>
+      <mass value="0.001"/> <inertia ixx="0.000001" ixy="0" ixz="0" iyy="0.000001" iyz="0" izz="0.000001"/>
+    </inertial>
+  </link>
+  <joint name="tof_joint" type="fixed">
+    <parent link="camera_link"/>
+    <child link="tof_link"/>
+    <origin xyz="0.025 0.0 -0.023" rpy="0 0 0"/>
+  </joint>
+  <gazebo reference="tof_link">
+    <sensor type="ray" name="tof_sensor">
+      <always_on>true</always_on>
+      <pose>0 0 0 0 0 0</pose>
+      <visualize>true</visualize> <update_rate>30</update_rate> <ray>
+        <scan>
+          <horizontal>
+            <samples>1</samples>
+            <resolution>1</resolution>
+            <min_angle>-0.01</min_angle> <max_angle>0.01</max_angle>
+          </horizontal>
+          <vertical>
+            <samples>1</samples>
+            <resolution>1</resolution>
+            <min_angle>-0.01</min_angle>
+            <max_angle>0.01</max_angle>
+          </vertical>
+        </scan>
+        <range>
+          <min>0.02</min> <max>2.0</max>  <resolution>0.01</resolution>
+        </range>
+        <radiation_type>infrared</radiation_type>
+      </ray>
+      <plugin name="tof_controller" filename="libgazebo_ros_ray_sensor.so">
+        <ros>
+          <namespace>/gimbal</namespace>
+          <remapping>~/out:=tof_distance</remapping>
+        </ros>
+        <output_type>sensor_msgs/LaserScan</output_type>
+        <radiation_type>infrared</radiation_type>
+        <frame_name>tof_link</frame_name>
+      </plugin>
+    </sensor>
+  </gazebo>
 </robot>
